File: hw-12v/door_light.sch (EAGLE design)
At the start: 24 parts, among them IC1 TINY13-20SSU, IC2 78L05F, T1 IRFML8244, T2 IRFML8244, T3 KP-3216P3C

Commit message: recalculated some resitors values
Parts:
- R2: value 470R -> 180R
- R7, R9: value 2.9kR -> 2.7kR
Changed lines of the file:
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@@
 <part name="F1" library="rcl" deviceset="R-EU_" device="MELF0204W" value="F750mA"/>
 <part name="R5" library="rcl" deviceset="R-EU_" device="R0402" value="10kR"/>
-<part name="R7" library="rcl" deviceset="R-EU_" device="R0603" value="2.9kR"/>
+<part name="R7" library="rcl" deviceset="R-EU_" device="R0603" value="2.7kR"/>
 <part name="R8" library="rcl" deviceset="R-EU_" device="R0603" value="10kR"/>
 <part name="R6" library="rcl" deviceset="R-EU_" device="R0603" value="10kR"/>
-<part name="R9" library="rcl" deviceset="R-EU_" device="R0603" value="2.9kR"/>
+<part name="R9" library="rcl" deviceset="R-EU_" device="R0603" value="2.7kR"/>
 <part name="SUPPLY24" library="supply2" deviceset="0V" device=""/>
 <part name="SUPPLY25" library="supply2" deviceset="0V" device=""/>
 <part name="LED2" library="led" deviceset="LED" device="CHIPLED_1206" value="IR"/>
 <part name="LED1" library="led" deviceset="LED" device="CHIPLED_0603" value="RED"/>
-<part name="R2" library="rcl" deviceset="R-EU_" device="R0603" value="470R"/>
+<part name="R2" library="rcl" deviceset="R-EU_" device="R0603" value="180R"/>
 <part name="R1" library="rcl" deviceset="R-EU_" device="R0603" value="470R"/>
 <part name="T3" library="opto-trans-smd" deviceset="KP-3216P3C" device=""/>

Commit message: fixed R5 size (was 40x should be 603)
Parts:
- R5: device rcl:R-EU_R0402 -> rcl:R-EU_R0603
Changed lines of the file:
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@@
 <part name="SUPPLY19" library="supply2" deviceset="0V" device=""/>
 <part name="F1" library="rcl" deviceset="R-EU_" device="MELF0204W" value="F750mA"/>
-<part name="R5" library="rcl" deviceset="R-EU_" device="R0402" value="10kR"/>
+<part name="R5" library="rcl" deviceset="R-EU_" device="R0603" value="10kR"/>
 <part name="R7" library="rcl" deviceset="R-EU_" device="R0603" value="2.7kR"/>
 <part name="R8" library="rcl" deviceset="R-EU_" device="R0603" value="10kR"/>

Commit message: fuse changed from 750mA to 350mA
Parts:
- F1: value F750mA -> F350mA
Changed lines of the file:
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@@
 <part name="C1" library="rcl" deviceset="C-EU" device="C1206" value="100nF"/>
 <part name="SUPPLY19" library="supply2" deviceset="0V" device=""/>
-<part name="F1" library="rcl" deviceset="R-EU_" device="MELF0204W" value="F750mA"/>
+<part name="F1" library="rcl" deviceset="R-EU_" device="MELF0204W" value="F350mA"/>
 <part name="R5" library="rcl" deviceset="R-EU_" device="R0603" value="10kR"/>
 <part name="R7" library="rcl" deviceset="R-EU_" device="R0603" value="2.7kR"/>
